Commit message: Completed URDF Tutorial

File: src/kh4_description/sdf/kh4.urdf (robot description, URDF)
Before this commit: robot kh4_robot, 3 links, 2 joints
Links:
- removed link kh4_robot__left_wheel
- removed link kh4_robot__right_wheel
- removed link kh4_robot_chassis
- added link chassis; collision cylinder length=.053 radius=.0704; collision sphere radius=.0047
- added link chassis_inertia, mass 0.5
- added link left_wheel, mass 0.033; collision cylinder length=0.005 radius=0.021; visual cylinder length=0.005 radius=0.021
- added link right_wheel, mass 0.033; collision cylinder length=0.005 radius=0.021; visual cylinder length=0.005 radius=0.021
Joints:
- removed joint kh4_robot__left_wheel_hinge
- removed joint kh4_robot__right_wheel_hinge
- added joint chassis_inertia_joint: type fixed, parent chassis, child chassis_inertia, origin xyz=0 0 0 rpy=0 0 0, axis 0 0 0
- added joint left_wheel_joint: type continuous, parent chassis, child left_wheel, origin xyz=0 0 0 rpy=0 0 0, axis 0 0 1
- added joint right_wheel_joint: type continuous, parent chassis, child right_wheel, origin xyz=0 0 0 rpy=0 0 0, axis 0 0 1

Commit message: base_link added

File: src/kh4_description/sdf/kh4.urdf (robot description, URDF)
Before this commit: robot kh4_robot, 4 links, 3 joints
Links:
- removed link chassis
- added link base_link; collision cylinder length=.053 radius=.0704; collision sphere radius=.0047
Joints:
- joint chassis_inertia_joint: parent chassis -> base_link
- joint left_wheel_joint: parent chassis -> base_link
- joint right_wheel_joint: parent chassis -> base_link

Commit message: URDF model. Missing <gazebo> tags

File: src/kh4_description/sdf/kh4.urdf (robot description, URDF)
Before this commit: robot kh4_robot, 4 links, 3 joints
Joints:
- joint left_wheel_joint: axis 0 0 1 -> 0 1 0; origin xyz=0 0 0 rpy=0 0 0 -> xyz=0 0.0527 -0.0102 rpy=0 0 0
- joint right_wheel_joint: axis 0 0 1 -> 0 1 0; origin xyz=0 0 0 rpy=0 0 0 -> xyz=0 -0.0527 -0.0102 rpy=0 0 0

Commit message: Added IMU and IR sensors

File: src/kh4_description/sdf/kh4.urdf (robot description, URDF)
Before this commit: robot kh4_robot, 4 links, 3 joints
Links:
- added link IR_link, mass 1e-5
- added link imu_link, mass 1e-5
Joints:
- added joint IR_joint: type fixed, parent base_link, child IR_link, origin xyz=0 0 0 rpy=0 0 0, axis 0 0 1
- added joint imu_joint: type fixed, parent base_link, child imu_link, origin xyz=0 0 0 rpy=0 0 0, axis 0 0 1

Commit message: Added sonars

File: src/kh4_description/sdf/kh4.urdf (robot description, URDF)
Before this commit: robot kh4_robot, 6 links, 5 joints
Links:
- added link sonar_link, mass 1e-5
Joints:
- added joint sonar_joint: type fixed, parent base_link, child sonar_link, origin xyz=0 0 0 rpy=0 0 0, axis 0 0 1
