Commit message: Added camera

File: src/kh4_description/sdf/robot1_kh4.urdf (robot description, URDF)
Before this commit: robot kh4_robot, 7 links, 6 joints
Links:
- added link camera_link; visual box size=0.02 0.02 0.02
Joints:
- added joint camera_joint: type fixed, parent base_link, child camera_link, origin xyz=.0704 0 0 rpy=0 0 0, axis 0 1 0
